Commit message: Bring up real hardware: standalone FollowJointTrajectory bridge, bypass ros2_control
ros2_control_node segfaults loading JointTrajectoryController on this setup, so
canbus_bridge.py is now a standalone ROS 2 node that is itself the robot driver:
runs the startup/homing sequence, publishes /joint_states from live encoders, and
serves a FollowJointTrajectory action server that MoveIt talks to directly via
moveit_simple_controller_manager. demo.launch.py now starts robot_state_publisher +
move_group + RViz + the bridge, no ros2_control_node or spawners.

Also fixes found bringing up all 6 joints on real hardware:
- moveit_controllers.yaml was missing the required action_ns parameter, which
  made moveit_simple_controller_manager silently see zero usable controllers.
- URDF rest-pose rotation offset on J1/J4 so joint=0 matches the physical home
  chosen for wiring constraints (previously only matched the CAD export).
- Direction signs for J1-J3 verified and flipped from the doc's predictions.
- J3 verified as an asymmetric range (-45..+405 deg), not symmetric +-180.
- Wrist differential mixing sign (s6) verified and flipped.
- joint_limits.yaml given real position/velocity limits derived from the
  boards' flashed speed ceiling, instead of the placeholder 2.0 rad/s default.

File: robo_arm_moveit_config/config/robo_arm_simplified_for_urdf_v2_1.ros2_control.xacro (robot description, xacro)
@@ -6,5 +6,7 @@
             <hardware>
                 <!-- By default, set up controllers for simulation. This won't work on real hardware -->
-                <plugin>mock_components/GenericSystem</plugin>
+                <plugin>topic_based_ros2_control/TopicBasedSystem</plugin>
+                <param name="joint_commands_topic">/isaac_joint_commands</param>
+                <param name="joint_states_topic">/isaac_joint_states</param>
             </hardware>
             <joint name="revolute_1">

File: robo_arm_simplified_for_urdf_v2_1/urdf/robo_arm_simplified_for_urdf_v2_1.urdf (robot description, URDF)
Before this commit: robot robo_arm_simplified_for_urdf_v2_1, 12 links, 11 joints
Joints:
- joint revolute_1: origin xyz=-1.49235e-17 7.11621e-24 0.1037 rpy=0 -0 0 -> xyz=-1.49235e-17 7.11621e-24 0.1037 rpy=0 0 -1.570796
- joint revolute_4: origin xyz=3.9942e-16 -0.0404996 0.0353704 rpy=1.5708 2.36656e-17 1.75506e-29 -> xyz=3.9942e-16 -0.0404996 0.0353704 rpy=1.570796 0 -1.570796
