Commit message: Add multi-waypoint sequencer GUI, fix motion planning bugs found during testing
- Fix motor_to_joint_rad/wrist_forward: boards report real multi-revolution
  position directly, not a wrapped single-turn value - the old wrap_deg call
  silently corrupted readback (both /joint_states and arrival checks) for any
  joint move bigger than a fraction of a motor revolution
- Convert revolute_1/3/4/6 from continuous to revolute with real URDF limits -
  continuous joints were planning/interpolating in a wraparound space
- Correct J1's real safe range to -135/+210deg (asymmetric, wiring constraint)
- Add config/ompl_planning.yaml: tighten longest_valid_segment_fraction so
  OMPL's search can't hand over a path the final collision check would reject
- Fix moveit_controllers.yaml execution-duration-monitoring params (needed
  nesting under trajectory_execution:, not bare top-level keys)
- canbus_bridge.py: execution_lock so only one trajectory drives the motors
  at a time, real arrival verification instead of trusting elapsed time,
  downsampled intermediate waypoint sends
- Add arm_driver/waypoint_gui.py: companion Tkinter app for building and
  running multi-waypoint sequences with per-segment velocity/wait, save/load
  named sequences, launches automatically with demo.launch.py
- Move one-off hardware diagnostic scripts into arm_driver/diagnostics/

File: robo_arm_simplified_for_urdf_v2_1/urdf/robo_arm_simplified_for_urdf_v2_1.urdf (robot description, URDF)
Before this commit: robot robo_arm_simplified_for_urdf_v2_1, 12 links, 11 joints
Joints:
- joint revolute_1: limit (none) -> lower=-2.356194 upper=3.665191 effort=1 velocity=1; type continuous -> revolute
- joint revolute_3: limit (none) -> lower=-0.785398 upper=7.068583 effort=1 velocity=1; type continuous -> revolute
- joint revolute_4: limit (none) -> lower=-3.141593 upper=3.141593 effort=1 velocity=1; type continuous -> revolute
- joint revolute_6: limit (none) -> lower=-3.141593 upper=3.141593 effort=1 velocity=1; type continuous -> revolute
